Commit message: Update quadrotor_with_kinect_with_hokuyo_utm30lx.xacro
Kinect camera orientation changed

File: src/kubot_launch/urdf/quadrotor_with_kinect_with_hokuyo_utm30lx.xacro (robot description, xacro)
@@ -14,5 +14,5 @@
     <xacro:include filename="$(find hector_sensors_description)/urdf/kinect_camera.urdf.xacro" />
     <xacro:kinect_camera name="camera" parent="base_link">
-      <origin xyz="0.05 0.0 -0.06" rpy="0 0 0"/>
+      <origin xyz="0.0 0.0 -0.15" rpy="0 1 1"/>
     </xacro:kinect_camera>
 </robot>

Commit message: Camera rotaion and position corrected

File: src/kubot_launch/urdf/quadrotor_with_kinect_with_hokuyo_utm30lx.xacro (robot description, xacro)
@@ -1,5 +1,6 @@
 <?xml version="1.0"?>
 <robot name="quadrotor" xmlns:xacro="http://www.ros.org/wiki/xacro">
-    <xacro:property name="M_PI" value="3.1415926535897931" />
+    <xacro:property name="M_PI" value="3.1415926535897931" />   <!-- 90 degree -->
+    <xacro:property name="M_PI/4" value="0.78539816339" />      <!-- 45 degree -->
     <!-- Included URDF Files -->
     <xacro:include filename="$(find hector_quadrotor_description)/urdf/quadrotor_base.urdf.xacro" />
@@ -11,8 +12,8 @@
       <origin xyz="0.0 0.0 -0.097" rpy="${M_PI} 0 0"/>
     </xacro:hokuyo_utm30lx>
-        <!-- Kinect -->
+    <!-- Kinect -->
     <xacro:include filename="$(find hector_sensors_description)/urdf/kinect_camera.urdf.xacro" />
     <xacro:kinect_camera name="camera" parent="base_link">
-      <origin xyz="0.0 0.0 -0.15" rpy="0 1 1"/>
+      <origin xyz="0.1 0.0 -0.05" rpy="0 1 0"/>
     </xacro:kinect_camera>
 </robot>
